Commit message: fix

File: src/salt_pkg/urdf/zed_integration.xacro (robot description, xacro)
@@ -11,4 +11,9 @@
     <!-- Camera mounting point (the threaded screw hole in the bottom) -->
     <link name="zedm_camera_link"> </link>
+    <joint name="zed_camera_joint" type="fixed">
+        <parent link="base_link"/>
+        <child link="zedm_camera_link" />
+        <origin xyz="0 0 0" rpy="0 0 0"/>
+    </joint>
     <!-- Camera Center -->
     <link name="zedm_camera_center">
