Commit message: it drivesros2 topic list! did a lot of stuff to make that happen

File: src/salt_pkg/urdf/robot_model.xacro (robot description, xacro)
@@ -1,5 +1,12 @@
 <?xml version="1.0"?>
 <robot name="saltbot" xmlns:xacro="http://ros.org/wiki/xacro">
+    <xacro:include filename="/home/seniorproject/nvi_ws/install/salt_pkg/share/salt_pkg/urdf/gazebo_ref.xacro" />
+    <xacro:include filename="/home/seniorproject/nvi_ws/install/salt_pkg/share/salt_pkg/urdf/gazebo_control.xacro" />
     <xacro:include filename="/home/seniorproject/nvi_ws/install/salt_pkg/share/salt_pkg/urdf/materials.xacro" />
+    <xacro:property name="base_length" value=".762"/>
+    <xacro:property name="base_width" value=".5334"/>
+    <xacro:property name="base_height" value=".2"/>
+    <xacro:property name="wheel_radius" value=".11"/>
+    <xacro:property name="wheel_width" value=".04"/>
     <link name="base_footprint"/>
     <joint name="base_joint" type="fixed">
@@ -12,5 +19,5 @@
             <origin xyz="0 0 .21" rpy="0 0 0"/>
             <geometry>
-                <box size=".762 .5334 .2"/>
+                <box size="${base_length} ${base_width} ${base_height}"/>
             </geometry>
             <material name="grey"/>
@@ -19,12 +26,57 @@
             <origin xyz="0 0 0.21" rpy="0 0 0"/>
             <geometry>
-                <box size=".762 .5334 .2"/>
+                <box size="${base_length} ${base_width} ${base_height}"/>
             </geometry>
         </collision>
+        <xacro:box_inertia m="15" w="${base_width}" d="${base_length}" h="${base_height}"/>
+    </link>
+    <joint name="left_wheel_joint" type="continuous">
+        <parent link="base_link"/>
+        <child link="left_wheel_link"/>
+        <origin xyz="0 0.271 .1" rpy="-1.57 0 0"/>
+        <axis xyz="0 0 1"/>
+    </joint>
+    <link name="left_wheel_link">
+        <visual>
+            <origin xyz="0 0 0" rpy="0 0 1.57"/>
+            <geometry>
+                <cylinder radius="${wheel_radius}" length="${wheel_width}"/>
+            </geometry>
+            <material name="red"/>
+        </visual>
+        <collision>
+            <origin xyz="0 0 0" rpy="0 0 1.57"/>
+            <geometry>
+                <cylinder radius="${wheel_radius}" length="${wheel_width}"/>
+            </geometry>
+        </collision>
+        <xacro:cylinder_inertia m="0.5" r="${wheel_radius}" h="${wheel_width}"/>
+    </link>
+    <joint name="right_wheel_joint" type="continuous">
+        <parent link="base_link"/>
+        <child link="right_wheel_link"/>
+        <origin xyz="0 -0.271 .1" rpy="-1.57 0 0"/>
+        <axis xyz="0 0 1"/>
+    </joint>
+    <link name="right_wheel_link">
+        <visual>
+            <origin xyz="0 0 0" rpy="0 0 1.57"/>
+            <geometry>
+                <cylinder radius="${wheel_radius}" length="${wheel_width}"/>
+            </geometry>
+            <material name="red"/>
+        </visual>
+        <collision>
+            <origin xyz="0 0 0" rpy="0 0 1.57"/>
+            <geometry>
+                <cylinder radius="${wheel_radius}" length="${wheel_width}"/>
+            </geometry>
+        </collision>
+        <xacro:cylinder_inertia m="0.5" r="${wheel_radius}" h="${wheel_width}"/>
     </link>
     <joint name="BRwheel_joint" type="continuous">
         <parent link="base_link"/>
         <child link="BRwheel_link"/>
-        <origin xyz="-.2667 -0.271 .1" rpy="-1.57 0 0"/>
+        <origin xyz="-.2667 -0.271 .103" rpy="-1.57 0 0"/>
         <axis xyz="0 0 1"/>
     </joint>
@@ -33,19 +85,14 @@
             <origin xyz="0 0 0" rpy="0 0 1.57"/>
             <geometry>
-                <cylinder length="0.04" radius="0.11"/>
+                <cylinder radius="${wheel_radius}" length="${wheel_width}"/>
             </geometry>
             <material name="red"/>
         </visual>
-        <collision>
-            <origin xyz="0 0 0" rpy="0 0 1.57"/>
-            <geometry>
-                <cylinder length="0.04" radius="0.11"/>
-            </geometry>
-        </collision>
+        <xacro:cylinder_inertia m="0.5" r="${wheel_radius}" h="${wheel_width}"/>
     </link>
     <joint name="FRwheel_joint" type="continuous">
         <parent link="base_link"/>
         <child link="FRwheel_link"/>
-        <origin xyz=".2667 -0.271 .1" rpy="-1.57 0 0"/>
+        <origin xyz=".2667 -0.271 .103" rpy="-1.57 0 0"/>
         <axis xyz="0 0 1"/>
     </joint>
@@ -54,19 +101,14 @@
             <origin xyz="0 0 0" rpy="0 0 1.57"/>
             <geometry>
-                <cylinder length="0.04" radius="0.11"/>
+                <cylinder radius="${wheel_radius}" length="${wheel_width}"/>
             </geometry>
             <material name="green"/>
         </visual>
-        <collision>
-            <origin xyz="0 0 0" rpy="0 0 1.57"/>
-            <geometry>
-                <cylinder length="0.04" radius="0.11"/>
-            </geometry>
-        </collision>
+        <xacro:cylinder_inertia m="0.5" r="${wheel_radius}" h="${wheel_width}"/>
     </link>
     <joint name="BLwheel_joint" type="continuous">
         <parent link="base_link"/>
         <child link="BLwheel_link"/>
-        <origin xyz="-.2667 0.271 .1" rpy="-1.57 0 0"/>
+        <origin xyz="-.2667 0.271 .103" rpy="-1.57 0 0"/>
         <axis xyz="0 0 1"/>
     </joint>
@@ -75,19 +117,14 @@
             <origin xyz="0 0 0" rpy="0 0 1.57"/>
             <geometry>
-                <cylinder length="0.04" radius="0.11"/>
+                <cylinder radius="${wheel_radius}" length="${wheel_width}"/>
             </geometry>
             <material name="orange"/>
         </visual>
-        <collision>
-            <origin xyz="0 0 0" rpy="0 0 1.57"/>
-            <geometry>
-                <cylinder length="0.04" radius="0.11"/>
-            </geometry>
-        </collision>
+        <xacro:cylinder_inertia m="0.5" r="${wheel_radius}" h="${wheel_width}"/>
     </link>
     <joint name="FLwheel_joint" type="continuous">
         <parent link="base_link"/>
         <child link="FLwheel_link"/>
-        <origin xyz=".2667 0.271 .1" rpy="-1.57 0 0"/>
+        <origin xyz=".2667 0.271 .103" rpy="-1.57 0 0"/>
         <axis xyz="0 0 1"/>
     </joint>
@@ -96,14 +133,57 @@
             <origin xyz="0 0 0" rpy="0 0 1.57"/>
             <geometry>
-                <cylinder length="0.04" radius="0.11"/>
+                <cylinder radius="${wheel_radius}" length="${wheel_width}"/>
             </geometry>
             <material name="blue"/>
         </visual>
+        <xacro:cylinder_inertia m="0.5" r="${wheel_radius}" h="${wheel_width}"/>
+    </link>
+    <joint name="imu_joint" type="fixed">
+        <parent link="base_link"/>
+        <child link="imu_link"/>
+        <origin xyz=".3 0 .325"/>
+    </joint>
+    <link name="imu_link">
+        <visual>
+            <geometry>
+                <box size="0.1 0.1 0.05"/>
+            </geometry>
+        </visual>
         <collision>
-            <origin xyz="0 0 0" rpy="0 0 1.57"/>
             <geometry>
-                <cylinder length="0.04" radius="0.11"/>
+                <box size="0.1 0.1 0.05"/>
             </geometry>
         </collision>
+        <xacro:box_inertia m="0.1" w="0.1" d="0.1" h="0.1"/>
     </link>
+    <link name="camera_link">
+        <visual>
+            <origin xyz="0 0 0" rpy="0 0 0"/>
+            <geometry>
+                <box size="0.015 0.015 0.5"/>
+            </geometry>
+        </visual>
+        <collision>
+            <origin xyz="0 0 0" rpy="0 0 0"/>
+            <geometry>
+                <box size="0.015 0.130 0.022"/>
+            </geometry>
+        </collision>
+        <inertial>
+            <origin xyz="0 0 0" rpy="0 0 0"/>
+            <mass value="0.035"/>
+            <inertia ixx="0.001"  ixy="0"  ixz="0" iyy="0.001" iyz="0" izz="0.001" />
+        </inertial>
+    </link>
+    <joint name="camera_joint" type="fixed">
+        <parent link="base_link"/>
+        <child link="camera_link"/>
+        <origin xyz=".3 0 .325"/>
+    </joint>
+    <link name="camera_depth_frame"/>
+    <joint name="camera_depth_joint" type="fixed">
+        <origin xyz="0 0 0" rpy="${-pi/2} 0 ${-pi/2}"/>
+        <parent link="camera_link"/>
+        <child link="camera_depth_frame"/>
+    </joint>
 </robot>

Commit message: gazebo simulation works without nav2 plugins

File: src/salt_pkg/urdf/robot_model.xacro (robot description, xacro)
@@ -8,4 +8,5 @@
     <xacro:property name="base_height" value=".2"/>
     <xacro:property name="wheel_radius" value=".11"/>
+    <xacro:property name="secondary_wheel_radius" value=".108"/>
     <xacro:property name="wheel_width" value=".04"/>
     <link name="base_footprint"/>
@@ -85,9 +86,15 @@
             <origin xyz="0 0 0" rpy="0 0 1.57"/>
             <geometry>
-                <cylinder radius="${wheel_radius}" length="${wheel_width}"/>
+                <cylinder radius="${secondary_wheel_radius}" length="${wheel_width}"/>
             </geometry>
             <material name="red"/>
         </visual>
-        <xacro:cylinder_inertia m="0.5" r="${wheel_radius}" h="${wheel_width}"/>
+        <collision>
+            <origin xyz="0 0 0" rpy="0 0 1.57"/>
+            <geometry>
+                <cylinder length="0.04" radius="0.11"/>
+            </geometry>
+        </collision>
+        <xacro:cylinder_inertia m="0.5" r="${secondary_wheel_radius}" h="${wheel_width}"/>
     </link>
     <joint name="FRwheel_joint" type="continuous">
@@ -101,9 +108,15 @@
             <origin xyz="0 0 0" rpy="0 0 1.57"/>
             <geometry>
-                <cylinder radius="${wheel_radius}" length="${wheel_width}"/>
+                <cylinder radius="${secondary_wheel_radius}" length="${wheel_width}"/>
             </geometry>
             <material name="green"/>
         </visual>
-        <xacro:cylinder_inertia m="0.5" r="${wheel_radius}" h="${wheel_width}"/>
+        <collision>
+            <origin xyz="0 0 0" rpy="0 0 1.57"/>
+            <geometry>
+                <cylinder length="0.04" radius="0.11"/>
+            </geometry>
+        </collision>
+        <xacro:cylinder_inertia m="0.5" r="${secondary_wheel_radius}" h="${wheel_width}"/>
     </link>
     <joint name="BLwheel_joint" type="continuous">
@@ -117,9 +130,15 @@
             <origin xyz="0 0 0" rpy="0 0 1.57"/>
             <geometry>
-                <cylinder radius="${wheel_radius}" length="${wheel_width}"/>
+                <cylinder radius="${secondary_wheel_radius}" length="${wheel_width}"/>
             </geometry>
             <material name="orange"/>
         </visual>
-        <xacro:cylinder_inertia m="0.5" r="${wheel_radius}" h="${wheel_width}"/>
+        <collision>
+            <origin xyz="0 0 0" rpy="0 0 1.57"/>
+            <geometry>
+                <cylinder length="0.04" radius="0.11"/>
+            </geometry>
+        </collision>
+        <xacro:cylinder_inertia m="0.5" r="${secondary_wheel_radius}" h="${wheel_width}"/>
     </link>
     <joint name="FLwheel_joint" type="continuous">
@@ -133,9 +152,15 @@
             <origin xyz="0 0 0" rpy="0 0 1.57"/>
             <geometry>
-                <cylinder radius="${wheel_radius}" length="${wheel_width}"/>
+                <cylinder radius="${secondary_wheel_radius}" length="${wheel_width}"/>
             </geometry>
             <material name="blue"/>
         </visual>
-        <xacro:cylinder_inertia m="0.5" r="${wheel_radius}" h="${wheel_width}"/>
+        <collision>
+            <origin xyz="0 0 0" rpy="0 0 1.57"/>
+            <geometry>
+                <cylinder length="0.04" radius="0.11"/>
+            </geometry>
+        </collision>
+        <xacro:cylinder_inertia m="0.5" r="${secondary_wheel_radius}" h="${wheel_width}"/>
     </link>
     <joint name="imu_joint" type="fixed">

Commit message: xacro doesnt work on zed_macro, idk how to install depth camera yet

File: src/salt_pkg/urdf/robot_model.xacro (robot description, xacro)
@@ -10,4 +10,9 @@
     <xacro:property name="secondary_wheel_radius" value=".108"/>
     <xacro:property name="wheel_width" value=".04"/>
+    <xacro:arg name="camera_name"   default="zedm" />
+    <xacro:arg name="camera_model"  default="zedm" />
+    <xacro:arg name="use_zed_localization" default="true" />
+    <xacro:include filename="$(find zed_wrapper)/urdf/zed_macro.urdf.xacro" />
+    <xacro:zed_camera name="$(arg camera_name)" model="$(arg camera_model)" />
     <link name="base_footprint"/>
     <joint name="base_joint" type="fixed">
@@ -182,5 +187,5 @@
         <xacro:box_inertia m="0.1" w="0.1" d="0.1" h="0.1"/>
     </link>
-    <link name="camera_link">
+    <link name="$(arg camera_name)_camera_link">
         <visual>
             <origin xyz="0 0 0" rpy="0 0 0"/>
@@ -201,14 +206,12 @@
         </inertial>
     </link>
-    <joint name="camera_joint" type="fixed">
-        <parent link="base_link"/>
-        <child link="camera_link"/>
-        <origin xyz=".3 0 .325"/>
-    </joint>
-    <link name="camera_depth_frame"/>
-    <joint name="camera_depth_joint" type="fixed">
-        <origin xyz="0 0 0" rpy="${-pi/2} 0 ${-pi/2}"/>
-        <parent link="camera_link"/>
-        <child link="camera_depth_frame"/>
+    <!-- ZED Localization -> The reference link is '$(arg camera_name)_camera_link' and 'base_link' is a child -->
+    <joint name="$(arg camera_name)_joint" type="fixed">
+      <parent link="$(arg camera_name)_camera_link"/>
+      <child link="base_link"/>
+      <origin
+        xyz="-0.12 0.0 -0.25"
+        rpy="0 0 0"
+      />
     </joint>
 </robot>

Commit message: move stuff around

File: src/salt_pkg/urdf/robot_model.xacro (robot description, xacro)
@@ -1,6 +1,8 @@
 <?xml version="1.0"?>
 <robot name="saltbot" xmlns:xacro="http://ros.org/wiki/xacro">
+    <!--
     <xacro:include filename="/home/seniorproject/nvi_ws/install/salt_pkg/share/salt_pkg/urdf/gazebo_ref.xacro" />
     <xacro:include filename="/home/seniorproject/nvi_ws/install/salt_pkg/share/salt_pkg/urdf/gazebo_control.xacro" />
+    -->
     <xacro:include filename="/home/seniorproject/nvi_ws/install/salt_pkg/share/salt_pkg/urdf/materials.xacro" />
     <xacro:property name="base_length" value=".762"/>
@@ -13,6 +15,5 @@
     <xacro:arg name="camera_model"  default="zedm" />
     <xacro:arg name="use_zed_localization" default="true" />
-    <xacro:include filename="$(find zed_wrapper)/urdf/zed_macro.urdf.xacro" />
-    <xacro:zed_camera name="$(arg camera_name)" model="$(arg camera_model)" />
+    <xacro:include filename="/home/seniorproject/nvi_ws/install/salt_pkg/share/salt_pkg/urdf/zed_integration.xacro" />
     <link name="base_footprint"/>
     <joint name="base_joint" type="fixed">
@@ -35,5 +36,5 @@
             </geometry>
         </collision>
-        <xacro:box_inertia m="15" w="${base_width}" d="${base_length}" h="${base_height}"/>
+        <!--<xacro:box_inertia m="15" w="${base_width}" d="${base_length}" h="${base_height}"/>-->
     </link>
     <joint name="left_wheel_joint" type="continuous">
@@ -57,5 +58,5 @@
             </geometry>
         </collision>
-        <xacro:cylinder_inertia m="0.5" r="${wheel_radius}" h="${wheel_width}"/>
+        <!--<xacro:cylinder_inertia m="0.5" r="${wheel_radius}" h="${wheel_width}"/>-->
     </link>
     <joint name="right_wheel_joint" type="continuous">
@@ -79,5 +80,5 @@
             </geometry>
         </collision>
-        <xacro:cylinder_inertia m="0.5" r="${wheel_radius}" h="${wheel_width}"/>
+        <!--<xacro:cylinder_inertia m="0.5" r="${wheel_radius}" h="${wheel_width}"/>-->
     </link>
     <joint name="BRwheel_joint" type="continuous">
@@ -101,5 +102,5 @@
             </geometry>
         </collision>
-        <xacro:cylinder_inertia m="0.5" r="${secondary_wheel_radius}" h="${wheel_width}"/>
+        <!--<xacro:cylinder_inertia m="0.5" r="${secondary_wheel_radius}" h="${wheel_width}"/>-->
     </link>
     <joint name="FRwheel_joint" type="continuous">
@@ -123,5 +124,5 @@
             </geometry>
         </collision>
-        <xacro:cylinder_inertia m="0.5" r="${secondary_wheel_radius}" h="${wheel_width}"/>
+        <!--<xacro:cylinder_inertia m="0.5" r="${secondary_wheel_radius}" h="${wheel_width}"/>-->
     </link>
     <joint name="BLwheel_joint" type="continuous">
@@ -145,5 +146,5 @@
             </geometry>
         </collision>
-        <xacro:cylinder_inertia m="0.5" r="${secondary_wheel_radius}" h="${wheel_width}"/>
+        <!--<xacro:cylinder_inertia m="0.5" r="${secondary_wheel_radius}" h="${wheel_width}"/>-->
     </link>
     <joint name="FLwheel_joint" type="continuous">
@@ -167,5 +168,5 @@
             </geometry>
         </collision>
-        <xacro:cylinder_inertia m="0.5" r="${secondary_wheel_radius}" h="${wheel_width}"/>
+        <!--<xacro:cylinder_inertia m="0.5" r="${secondary_wheel_radius}" h="${wheel_width}"/>-->
     </link>
     <joint name="imu_joint" type="fixed">
@@ -185,33 +186,5 @@
             </geometry>
         </collision>
-        <xacro:box_inertia m="0.1" w="0.1" d="0.1" h="0.1"/>
+        <!--<xacro:box_inertia m="0.1" w="0.1" d="0.1" h="0.1"/>-->
     </link>
-    <link name="$(arg camera_name)_camera_link">
-        <visual>
-            <origin xyz="0 0 0" rpy="0 0 0"/>
-            <geometry>
-                <box size="0.015 0.015 0.5"/>
-            </geometry>
-        </visual>
-        <collision>
-            <origin xyz="0 0 0" rpy="0 0 0"/>
-            <geometry>
-                <box size="0.015 0.130 0.022"/>
-            </geometry>
-        </collision>
-        <inertial>
-            <origin xyz="0 0 0" rpy="0 0 0"/>
-            <mass value="0.035"/>
-            <inertia ixx="0.001"  ixy="0"  ixz="0" iyy="0.001" iyz="0" izz="0.001" />
-        </inertial>
-    </link>
-    <!-- ZED Localization -> The reference link is '$(arg camera_name)_camera_link' and 'base_link' is a child -->
-    <joint name="$(arg camera_name)_joint" type="fixed">
-      <parent link="$(arg camera_name)_camera_link"/>
-      <child link="base_link"/>
-      <origin
-        xyz="-0.12 0.0 -0.25"
-        rpy="0 0 0"
-      />
-    </joint>
 </robot>

File: src/salt_pkg/urdf/zed_integration.xacro (robot description, xacro)
@@ -1,26 +1,60 @@
 <?xml version="1.0"?>
-<robot xmlns:xacro="http://www.ros.org/wiki/xacro">
-    <!-- This file is unused -->
-    <xacro:if value="$(arg use_zed_localization)">
-    <!-- ZED Localization -> The reference link is '$(arg camera_name)_camera_link' and 'base_link' is a child -->
-    <joint name="$(arg camera_name)_joint" type="fixed">
-      <parent link="$(arg camera_name)_camera_link"/>
-      <child link="base_link"/>
-      <origin
-        xyz="-0.12 0.0 -0.25"
-        rpy="0 0 0"
-      />
+<robot xmlns:xacro="http://wiki.ros.org/xacro">
+  <xacro:include filename="$(find zed_wrapper)/urdf/include/materials.urdf.xacro" />
+  <xacro:property name="M_PI"     value="3.1415926535897931" />
+    <xacro:property name="baseline" value="0.06" />
+    <xacro:property name="height" value="0.0265" />
+    <xacro:property name="bottom_slope" value="0.0" />
+    <xacro:property name="screw_offset_x" value="0.0" />
+    <xacro:property name="screw_offset_z" value="0.0" />
+    <xacro:property name="optical_offset_x" value="0.0" />
+    <!-- Camera mounting point (the threaded screw hole in the bottom) -->
+    <link name="zedm_camera_link"> </link>
+    <!-- Camera Center -->
+    <link name="zedm_camera_center">
+        <visual>
+          <origin xyz="${screw_offset_x} 0 ${screw_offset_z}" rpy="0 0 0"/>
+          <geometry>
+            <mesh filename="package://zed_interfaces/meshes/zedm.stl" />
+          </geometry>
+          <material name="zedm_mat" />
+        </visual>
+        <collision>
+          <origin xyz="${screw_offset_x} 0 ${screw_offset_z}" rpy="0 0 0"/>
+          <geometry>
+            <mesh filename="package://zed_interfaces/meshes/zedm.stl" />
+          </geometry>
+        </collision>
+    </link>
+    <joint name="zedm_camera_center_joint" type="fixed">
+      <parent link="zedm_camera_link"/>
+      <child link="zedm_camera_center"/>
+      <origin xyz="0 0 ${height/2}" rpy="0 ${bottom_slope} 0" />
     </joint>
-  </xacro:if>
-  <xacro:unless value="$(arg use_zed_localization)">
-    <!-- NO ZED Localization -> '$(arg camera_name)_camera_link' is a child of 'base_link' -->
-    <joint name="$(arg camera_name)_joint" type="fixed">
-      <parent link="base_link"/>
-      <child link="$(arg camera_name)_camera_link"/>
-      <origin
-        xyz="0.12 0.0 0.25"
-        rpy="0 0 0"
-      />
+    <!-- Left Camera -->
+    <link name="zedm_left_camera_frame"> </link>
+    <joint name="zedm_left_camera_joint" type="fixed">
+      <parent link="zedm_camera_center"/>
+      <child link="zedm_left_camera_frame"/>
+      <origin xyz="${optical_offset_x} ${baseline/2} 0" rpy="0 0 0" />
     </joint>
-  </xacro:unless>
+    <link name="zedm_left_camera_optical_frame"> </link>
+    <joint name="zedm_left_camera_optical_joint" type="fixed">
+      <origin xyz="0 0 0" rpy="-${M_PI/2} 0.0 -${M_PI/2}"/>
+      <parent link="zedm_left_camera_frame"/>
+      <child link="zedm_left_camera_optical_frame"/>
+    </joint>
+    <!-- Right Camera -->
+    <link name="zedm_right_camera_frame"> </link>
+    <joint name="zedm_right_camera_joint" type="fixed">
+      <parent link="zedm_camera_center"/>
+      <child link="zedm_right_camera_frame"/>
+      <origin xyz="${optical_offset_x} -${baseline/2} 0" rpy="0 0 0" />
+    </joint>
+    <link name="zedm_right_camera_optical_frame"> </link>
+    <joint name="zedm_right_camera_optical_joint" type="fixed">
+      <origin xyz="0 0 0" rpy="-${M_PI/2} 0.0 -${M_PI/2}"/>
+      <parent link="zedm_right_camera_frame"/>
+      <child link="zedm_right_camera_optical_frame"/>
+    </joint>
 </robot>

Commit message: most recent

File: src/salt_pkg/urdf/robot_model.xacro (robot description, xacro)
@@ -17,5 +17,5 @@
     <xacro:include filename="/home/seniorproject/nvi_ws/install/salt_pkg/share/salt_pkg/urdf/zed_integration.xacro" />
     <link name="base_footprint"/>
-    <joint name="base_joint" type="fixed">
+    <joint name="base_footprint_joint" type="fixed">
         <parent link="base_footprint"/>
         <child link="base_link" />
