Commit message: IT WORKS

File: src/salt_pkg/urdf/robot_model.xacro (robot description, xacro)
@@ -15,12 +15,11 @@
     <xacro:arg name="camera_model"  default="zedm" />
     <xacro:arg name="use_zed_localization" default="true" />
-    <xacro:include filename="/home/seniorproject/nvi_ws/install/salt_pkg/share/salt_pkg/urdf/zed_integration.xacro" />
-    <link name="base_footprint"/>
-    <joint name="base_footprint_joint" type="fixed">
-        <parent link="base_footprint"/>
-        <child link="base_link" />
+    <link name="zed_camera_link"/>
+    <joint name="base_link_joint" type="fixed">
+        <parent link="zed_camera_link"/>
+        <child link="frame" />
         <origin xyz="0 0 0" rpy="0 0 0"/>
     </joint>
-    <link name="base_link">
+    <link name="frame">
         <visual>
             <origin xyz="0 0 .21" rpy="0 0 0"/>
@@ -39,5 +38,5 @@
     </link>
     <joint name="left_wheel_joint" type="continuous">
-        <parent link="base_link"/>
+        <parent link="frame"/>
         <child link="left_wheel_link"/>
         <origin xyz="0 0.271 .1" rpy="-1.57 0 0"/>
@@ -61,5 +60,5 @@
     </link>
     <joint name="right_wheel_joint" type="continuous">
-        <parent link="base_link"/>
+        <parent link="frame"/>
         <child link="right_wheel_link"/>
         <origin xyz="0 -0.271 .1" rpy="-1.57 0 0"/>
@@ -83,5 +82,5 @@
     </link>
     <joint name="BRwheel_joint" type="continuous">
-        <parent link="base_link"/>
+        <parent link="frame"/>
         <child link="BRwheel_link"/>
         <origin xyz="-.2667 -0.271 .103" rpy="-1.57 0 0"/>
@@ -105,5 +104,5 @@
     </link>
     <joint name="FRwheel_joint" type="continuous">
-        <parent link="base_link"/>
+        <parent link="frame"/>
         <child link="FRwheel_link"/>
         <origin xyz=".2667 -0.271 .103" rpy="-1.57 0 0"/>
@@ -127,5 +126,5 @@
     </link>
     <joint name="BLwheel_joint" type="continuous">
-        <parent link="base_link"/>
+        <parent link="frame"/>
         <child link="BLwheel_link"/>
         <origin xyz="-.2667 0.271 .103" rpy="-1.57 0 0"/>
@@ -149,5 +148,5 @@
     </link>
     <joint name="FLwheel_joint" type="continuous">
-        <parent link="base_link"/>
+        <parent link="frame"/>
         <child link="FLwheel_link"/>
         <origin xyz=".2667 0.271 .103" rpy="-1.57 0 0"/>
@@ -171,5 +170,5 @@
     </link>
     <joint name="imu_joint" type="fixed">
-        <parent link="base_link"/>
+        <parent link="frame"/>
         <child link="imu_link"/>
         <origin xyz=".3 0 .325"/>

File: src/salt_pkg/urdf/zed_integration.xacro (robot description, xacro)
@@ -12,5 +12,5 @@
     <link name="zedm_camera_link"> </link>
     <joint name="zed_camera_joint" type="fixed">
-        <parent link="base_link"/>
+        <parent link="frame"/>
         <child link="zedm_camera_link" />
         <origin xyz="0 0 0" rpy="0 0 0"/>
